Commit message: added stick.xacro

File: urdf/stick.xacro (robot description, xacro)
@@ -1,33 +1,21 @@
 <?xml version="1.0"?>
-<robot name="builder_bot" xmlns:xacro="http://ros.org/wiki/xacro">
-    <xacro:arg name="bot_name" default="builder_bot" />
-    <xacro:include
-        filename="$(find builder_bot_description)/urdf/common_properties.xacro" />
-    <xacro:include
-        filename="$(find builder_bot_description)/urdf/builder_bot.gazebo" />
-    <link
-        name="base_footprint" />
-    <joint name="base_joint" type="fixed">
-        <parent link="base_footprint" />
-        <child link="base_link" />
-        <origin xyz="0.0 0.0 0.03" rpy="0 0 0" />
-    </joint>
+<robot name="multipleshapes">
     <link name="base_link">
         <visual>
-            <origin xyz="0.0 0.0 0.0" rpy="0 0 0" />
             <geometry>
+                <cylinder length="0.6" radius="0.2" />
             </geometry>
         </visual>
-        <collision>
-            <origin xyz="0.0 0.0 0.0 " rpy="0 0 0" />
+    </link>
+    <link name="right_leg">
+        <visual>
             <geometry>
-                <box size="0.1 0.08 0.02" />
+                <box size="0.6 0.1 0.2" />
             </geometry>
-        </collision>
-        <inertial>
-            <origin xyz="0.0 0.0 0.0" rpy="0 0 0" />
-            <mass value="2.75317" />
-            <inertia ixx="8.101e-03" ixy="0" ixz="0" iyy="6.775e-03" iyz="0" izz="9.798e-03" />
-        </inertial>
+        </visual>
     </link>
+    <joint name="base_to_right_leg" type="fixed">
+        <parent link="base_link" />
+        <child link="right_leg" />
+    </joint>
 </robot>

Commit message: demo xacro added

File: urdf/stick.xacro (robot description, xacro)
@@ -1,21 +1,195 @@
 <?xml version="1.0"?>
-<robot name="multipleshapes">
-    <link name="base_link">
+<!-- =================================================================================== -->
+<!-- |    This document was autogenerated by xacro from car-robot.xacro                | -->
+<!-- |    EDITING THIS FILE BY HAND IS NOT RECOMMENDED                                 | -->
+<!-- =================================================================================== -->
+<robot name="car-robot">
+    <!--dummy
+    link-->
+    <link name="base_link" />
+    <!--chassis
+    link-->
+    <link name="chassis-link">
         <visual>
+            <origin rpy="0 0 0" xyz="0 0 0" />
             <geometry>
-                <cylinder length="0.6" radius="0.2" />
+                <box size="0.14 0.12 0.01" />
             </geometry>
+            <material name="brown">
+                <color rgba="0.3 0 0.4 1" />
+            </material>
         </visual>
+        <collision>
+            <origin rpy="0 0 0" xyz="0 0 0" />
+            <geometry>
+                <box size="0.14 0.12 0.01" />
+            </geometry>
+        </collision>
+        <inertial>
+            <mass value="0.4" />
+            <inertia ixx="0.00048333" ixy="0" ixz="0" iyy="0.0013367" iyz="0" izz="0.0018133" />
+        </inertial>
     </link>
-    <link name="right_leg">
+    <joint name="joint-base-chassis" type="fixed">
+        <parent link="base_link" />
+        <child link="chassis-link" />
+        <origin rpy="0 0 0" xyz="0 0 0.02" />
+    </joint>
+    <material name="blue">
+        <color rgba="0 0.4 0.5 1" />
+    </material>
+    <!-- ${x_position}-${y_position}-wheel-link -->
+    <link name="front-right-wheel-link">
         <visual>
+            <origin rpy="1.5707963267948966 0 0" xyz="0 0 0" />
             <geometry>
-                <box size="0.6 0.1 0.2" />
+                <cylinder length="0.01" radius="0.02" />
             </geometry>
+            <material name="blue" />
         </visual>
+        <collision>
+            <origin rpy="1.5707963267948966 0 0" xyz="0 0 0" />
+            <geometry>
+                <cylinder length="0.01" radius="0.02" />
+            </geometry>
+        </collision>
+        <inertial>
+            <origin rpy="1.5707963267948966 0 0" xyz="0 0 0" />
+            <mass value="0.2" />
+            <inertia ixx="2.166666666666667e-05" ixy="0" ixz="0" iyy="2.166666666666667e-05" iyz="0"
+                izz="4e-05" />
+        </inertial>
     </link>
-    <joint name="base_to_right_leg" type="fixed">
-        <parent link="base_link" />
-        <child link="right_leg" />
+    <joint name="joint-chassis-front-right-wheel" type="continuous">
+        <parent link="chassis-link" />
+        <child link="front-right-wheel-link" />
+        <origin rpy="0 0 0" xyz="0.042 0.065 0" />
+        <axis xyz="0 1 0" />
     </joint>
+    <!-- ${x_position}-${y_position}-wheel-link -->
+    <link name="front-left-wheel-link">
+        <visual>
+            <origin rpy="1.5707963267948966 0 0" xyz="0 0 0" />
+            <geometry>
+                <cylinder length="0.01" radius="0.02" />
+            </geometry>
+            <material name="blue" />
+        </visual>
+        <collision>
+            <origin rpy="1.5707963267948966 0 0" xyz="0 0 0" />
+            <geometry>
+                <cylinder length="0.01" radius="0.02" />
+            </geometry>
+        </collision>
+        <inertial>
+            <origin rpy="1.5707963267948966 0 0" xyz="0 0 0" />
+            <mass value="0.2" />
+            <inertia ixx="2.166666666666667e-05" ixy="0" ixz="0" iyy="2.166666666666667e-05" iyz="0"
+                izz="4e-05" />
+        </inertial>
+    </link>
+    <joint name="joint-chassis-front-left-wheel" type="continuous">
+        <parent link="chassis-link" />
+        <child link="front-left-wheel-link" />
+        <origin rpy="0 0 0" xyz="0.042 -0.065 0" />
+        <axis xyz="0 1 0" />
+    </joint>
+    <!-- ${x_position}-${y_position}-wheel-link -->
+    <link name="rare-right-wheel-link">
+        <visual>
+            <origin rpy="1.5707963267948966 0 0" xyz="0 0 0" />
+            <geometry>
+                <cylinder length="0.01" radius="0.02" />
+            </geometry>
+            <material name="blue" />
+        </visual>
+        <collision>
+            <origin rpy="1.5707963267948966 0 0" xyz="0 0 0" />
+            <geometry>
+                <cylinder length="0.01" radius="0.02" />
+            </geometry>
+        </collision>
+        <inertial>
+            <origin rpy="1.5707963267948966 0 0" xyz="0 0 0" />
+            <mass value="0.2" />
+            <inertia ixx="2.166666666666667e-05" ixy="0" ixz="0" iyy="2.166666666666667e-05" iyz="0"
+                izz="4e-05" />
+        </inertial>
+    </link>
+    <joint name="joint-chassis-rare-right-wheel" type="continuous">
+        <parent link="chassis-link" />
+        <child link="rare-right-wheel-link" />
+        <origin rpy="0 0 0" xyz="-0.042 0.065 0" />
+        <axis xyz="0 1 0" />
+    </joint>
+    <!-- ${x_position}-${y_position}-wheel-link -->
+    <link name="rare-left-wheel-link">
+        <visual>
+            <origin rpy="1.5707963267948966 0 0" xyz="0 0 0" />
+            <geometry>
+                <cylinder length="0.01" radius="0.02" />
+            </geometry>
+            <material name="blue" />
+        </visual>
+        <collision>
+            <origin rpy="1.5707963267948966 0 0" xyz="0 0 0" />
+            <geometry>
+                <cylinder length="0.01" radius="0.02" />
+            </geometry>
+        </collision>
+        <inertial>
+            <origin rpy="1.5707963267948966 0 0" xyz="0 0 0" />
+            <mass value="0.2" />
+            <inertia ixx="2.166666666666667e-05" ixy="0" ixz="0" iyy="2.166666666666667e-05" iyz="0"
+                izz="4e-05" />
+        </inertial>
+    </link>
+    <joint name="joint-chassis-rare-left-wheel" type="continuous">
+        <parent link="chassis-link" />
+        <child link="rare-left-wheel-link" />
+        <origin rpy="0 0 0" xyz="-0.042 -0.065 0" />
+        <axis xyz="0 1 0" />
+    </joint>
+    <gazebo reference="chassis-link">
+        <material>Gazebo/DarkGrey</material>
+    </gazebo>
+    <gazebo>
+        <!-- differential drive control for Gazebo -->
+        <plugin filename="libgazebo_ros_diff_drive.so" name="differential_drive_controller">
+            <alwaysOn>true</alwaysOn>
+            <updateRate>100</updateRate>
+            <leftJoint>joint-chassis-rare-left-wheel</leftJoint>
+            <rightJoint>joint-chassis-rare-right-wheel</rightJoint>
+            <wheelSeparation>0.12</wheelSeparation>
+            <wheelDiameter>0.04</wheelDiameter>
+            <torque>0.1</torque>
+            <commandTopic>cmd_vel</commandTopic>
+            <odometryTopic>odom</odometryTopic>
+            <odometryFrame>odom</odometryFrame>
+            <robotBaseFrame>base_link</robotBaseFrame>
+            <publishWheelTF>true</publishWheelTF>
+            <publishOdom>true</publishOdom>
+            <publishWheelJointState>true</publishWheelJointState>
+        </plugin>
+    </gazebo>
+    <gazebo reference="front-right-wheel-link">
+        <mu1>10000.0 </mu1>
+        <mu2>10000.0 </mu2>
+        <material>Gazebo/Purple</material>
+    </gazebo>
+    <gazebo reference="front-left-wheel-link">
+        <mu1>10000.0 </mu1>
+        <mu2>10000.0 </mu2>
+        <material>Gazebo/Purple</material>
+    </gazebo>
+    <gazebo reference="rare-right-wheel-link">
+        <mu1>10000.0 </mu1>
+        <mu2>10000.0 </mu2>
+        <material>Gazebo/Purple</material>
+    </gazebo>
+    <gazebo reference="rare-left-wheel-link">
+        <mu1>10000.0 </mu1>
+        <mu2>10000.0 </mu2>
+        <material>Gazebo/Purple</material>
+    </gazebo>
 </robot>

Commit message: Tested demo urdf

File: urdf/stick.xacro (robot description, xacro)
@@ -1,18 +1,29 @@
-<?xml version="1.0"?>
-<!-- =================================================================================== -->
-<!-- |    This document was autogenerated by xacro from car-robot.xacro                | -->
-<!-- |    EDITING THIS FILE BY HAND IS NOT RECOMMENDED                                 | -->
-<!-- =================================================================================== -->
-<robot name="car-robot">
+<?xml version='1.0'?>
+<robot xmlns:xacro="http://www.ros.org/wiki/xacro" name="car_robot_chassis">
     <!--dummy
     link-->
+    <xacro:property name="chassis_length" value="0.14" />
+    <xacro:property name="chassis_width" value="0.12" />
+    <xacro:property name="chassis_height" value="0.01" />
+    <xacro:property name="chassis_mass" value="0.4" />
+    <xacro:property name="wheel_radius" value="0.02" />
+    <xacro:property name="wheel_height" value="0.01" />
+    <xacro:property name="wheel_mass" value="0.2" />
+    <!-- <xacro:macro name="box_inertia" params="mass L W H">
+        <inertia ixx="${1/12 * mass * (L**2 + W**2 )}" iyy="${1/12 * mass * (H**2 + W**2 )}"
+            izz="${1/12 * mass * (L**2 + H**2 )}"
+            ixy="0" ixz="0" iyz="0" />
+    </xacro:macro> -->
+    <xacro:macro name="cylinder_inertia" params="mass R H">
+        <inertia ixx="${1/12 * mass * (3 * R**2 + H**2 )}" iyy="${1/12 * mass * (3 * R**2 + H**2 )}"
+            izz="${0.5 * (mass * R**2 )}"
+            ixy="0" ixz="0" iyz="0" />
+    </xacro:macro>
     <link name="base_link" />
-    <!--chassis
-    link-->
     <link name="chassis-link">
         <visual>
-            <origin rpy="0 0 0" xyz="0 0 0" />
+            <origin xyz="0 0 0" rpy="0 0 0" />
             <geometry>
-                <box size="0.14 0.12 0.01" />
+                <box size="${chassis_length} ${chassis_width} ${chassis_height}" />
             </geometry>
             <material name="brown">
@@ -21,12 +32,13 @@
         </visual>
         <collision>
-            <origin rpy="0 0 0" xyz="0 0 0" />
+            <origin xyz="0 0 0" rpy="0 0 0" />
             <geometry>
-                <box size="0.14 0.12 0.01" />
+                <box size="${chassis_length} ${chassis_width} ${chassis_height}" />
             </geometry>
         </collision>
         <inertial>
             <mass value="0.4" />
-            <inertia ixx="0.00048333" ixy="0" ixz="0" iyy="0.0013367" iyz="0" izz="0.0018133" />
+            <inertia ixx="0.00048333" iyy="0.0013367" izz="0.0018133"
+                ixy="0" ixz="0" iyz="0" />
         </inertial>
     </link>
@@ -34,162 +46,43 @@
         <parent link="base_link" />
         <child link="chassis-link" />
-        <origin rpy="0 0 0" xyz="0 0 0.02" />
+        <origin xyz="0 0 ${wheel_radius}" rpy="0 0 0" />
     </joint>
     <material name="blue">
         <color rgba="0 0.4 0.5 1" />
     </material>
-    <!-- ${x_position}-${y_position}-wheel-link -->
-    <link name="front-right-wheel-link">
-        <visual>
-            <origin rpy="1.5707963267948966 0 0" xyz="0 0 0" />
-            <geometry>
-                <cylinder length="0.01" radius="0.02" />
-            </geometry>
-            <material name="blue" />
-        </visual>
-        <collision>
-            <origin rpy="1.5707963267948966 0 0" xyz="0 0 0" />
-            <geometry>
-                <cylinder length="0.01" radius="0.02" />
-            </geometry>
-        </collision>
-        <inertial>
-            <origin rpy="1.5707963267948966 0 0" xyz="0 0 0" />
-            <mass value="0.2" />
-            <inertia ixx="2.166666666666667e-05" ixy="0" ixz="0" iyy="2.166666666666667e-05" iyz="0"
-                izz="4e-05" />
-        </inertial>
-    </link>
-    <joint name="joint-chassis-front-right-wheel" type="continuous">
-        <parent link="chassis-link" />
-        <child link="front-right-wheel-link" />
-        <origin rpy="0 0 0" xyz="0.042 0.065 0" />
-        <axis xyz="0 1 0" />
-    </joint>
-    <!-- ${x_position}-${y_position}-wheel-link -->
-    <link name="front-left-wheel-link">
-        <visual>
-            <origin rpy="1.5707963267948966 0 0" xyz="0 0 0" />
-            <geometry>
-                <cylinder length="0.01" radius="0.02" />
-            </geometry>
-            <material name="blue" />
-        </visual>
-        <collision>
-            <origin rpy="1.5707963267948966 0 0" xyz="0 0 0" />
-            <geometry>
-                <cylinder length="0.01" radius="0.02" />
-            </geometry>
-        </collision>
-        <inertial>
-            <origin rpy="1.5707963267948966 0 0" xyz="0 0 0" />
-            <mass value="0.2" />
-            <inertia ixx="2.166666666666667e-05" ixy="0" ixz="0" iyy="2.166666666666667e-05" iyz="0"
-                izz="4e-05" />
-        </inertial>
-    </link>
-    <joint name="joint-chassis-front-left-wheel" type="continuous">
-        <parent link="chassis-link" />
-        <child link="front-left-wheel-link" />
-        <origin rpy="0 0 0" xyz="0.042 -0.065 0" />
-        <axis xyz="0 1 0" />
-    </joint>
-    <!-- ${x_position}-${y_position}-wheel-link -->
-    <link name="rare-right-wheel-link">
-        <visual>
-            <origin rpy="1.5707963267948966 0 0" xyz="0 0 0" />
-            <geometry>
-                <cylinder length="0.01" radius="0.02" />
-            </geometry>
-            <material name="blue" />
-        </visual>
-        <collision>
-            <origin rpy="1.5707963267948966 0 0" xyz="0 0 0" />
-            <geometry>
-                <cylinder length="0.01" radius="0.02" />
-            </geometry>
-        </collision>
-        <inertial>
-            <origin rpy="1.5707963267948966 0 0" xyz="0 0 0" />
-            <mass value="0.2" />
-            <inertia ixx="2.166666666666667e-05" ixy="0" ixz="0" iyy="2.166666666666667e-05" iyz="0"
-                izz="4e-05" />
-        </inertial>
-    </link>
-    <joint name="joint-chassis-rare-right-wheel" type="continuous">
-        <parent link="chassis-link" />
-        <child link="rare-right-wheel-link" />
-        <origin rpy="0 0 0" xyz="-0.042 0.065 0" />
-        <axis xyz="0 1 0" />
-    </joint>
-    <!-- ${x_position}-${y_position}-wheel-link -->
-    <link name="rare-left-wheel-link">
-        <visual>
-            <origin rpy="1.5707963267948966 0 0" xyz="0 0 0" />
-            <geometry>
-                <cylinder length="0.01" radius="0.02" />
-            </geometry>
-            <material name="blue" />
-        </visual>
-        <collision>
-            <origin rpy="1.5707963267948966 0 0" xyz="0 0 0" />
-            <geometry>
-                <cylinder length="0.01" radius="0.02" />
-            </geometry>
-        </collision>
-        <inertial>
-            <origin rpy="1.5707963267948966 0 0" xyz="0 0 0" />
-            <mass value="0.2" />
-            <inertia ixx="2.166666666666667e-05" ixy="0" ixz="0" iyy="2.166666666666667e-05" iyz="0"
-                izz="4e-05" />
-        </inertial>
-    </link>
-    <joint name="joint-chassis-rare-left-wheel" type="continuous">
-        <parent link="chassis-link" />
-        <child link="rare-left-wheel-link" />
-        <origin rpy="0 0 0" xyz="-0.042 -0.065 0" />
-        <axis xyz="0 1 0" />
-    </joint>
-    <gazebo reference="chassis-link">
-        <material>Gazebo/DarkGrey</material>
-    </gazebo>
-    <gazebo>
-        <!-- differential drive control for Gazebo -->
-        <plugin filename="libgazebo_ros_diff_drive.so" name="differential_drive_controller">
-            <alwaysOn>true</alwaysOn>
-            <updateRate>100</updateRate>
-            <leftJoint>joint-chassis-rare-left-wheel</leftJoint>
-            <rightJoint>joint-chassis-rare-right-wheel</rightJoint>
-            <wheelSeparation>0.12</wheelSeparation>
-            <wheelDiameter>0.04</wheelDiameter>
-            <torque>0.1</torque>
-            <commandTopic>cmd_vel</commandTopic>
-            <odometryTopic>odom</odometryTopic>
-            <odometryFrame>odom</odometryFrame>
-            <robotBaseFrame>base_link</robotBaseFrame>
-            <publishWheelTF>true</publishWheelTF>
-            <publishOdom>true</publishOdom>
-            <publishWheelJointState>true</publishWheelJointState>
-        </plugin>
-    </gazebo>
-    <gazebo reference="front-right-wheel-link">
-        <mu1>10000.0 </mu1>
-        <mu2>10000.0 </mu2>
-        <material>Gazebo/Purple</material>
-    </gazebo>
-    <gazebo reference="front-left-wheel-link">
-        <mu1>10000.0 </mu1>
-        <mu2>10000.0 </mu2>
-        <material>Gazebo/Purple</material>
-    </gazebo>
-    <gazebo reference="rare-right-wheel-link">
-        <mu1>10000.0 </mu1>
-        <mu2>10000.0 </mu2>
-        <material>Gazebo/Purple</material>
-    </gazebo>
-    <gazebo reference="rare-left-wheel-link">
-        <mu1>10000.0 </mu1>
-        <mu2>10000.0 </mu2>
-        <material>Gazebo/Purple</material>
-    </gazebo>
+    <xacro:macro name="wheel" params="x_position y_position x_reflect y_reflect">
+        <!-- ${x_position}-${y_position}-wheel-link -->
+        <link name="${x_position}-${y_position}-wheel-link">
+            <visual>
+                <origin xyz="0 0 0" rpy="${pi * 0.5} 0 0" />
+                <geometry>
+                    <cylinder radius="${wheel_radius}" length="${wheel_height}" />
+                </geometry>
+                <material name="blue" />
+            </visual>
+            <collision>
+                <origin xyz="0 0 0" rpy="${pi * 0.5} 0 0" />
+                <geometry>
+                    <cylinder radius="${wheel_radius}" length="${wheel_height}" />
+                </geometry>
+            </collision>
+            <inertial>
+                <origin xyz="0 0 0" rpy="${pi * 0.5} 0 0" />
+                <mass value="${wheel_mass}" />
+                <xacro:cylinder_inertia mass="${wheel_mass}" R="${wheel_radius}" H="${wheel_height}" />
+            </inertial>
+        </link>
+        <joint name="joint-chassis-${x_position}-${y_position}-wheel" type="continuous">
+            <parent link="chassis-link" />
+            <child link="${x_position}-${y_position}-wheel-link" />
+            <origin
+                xyz="${x_reflect*0.3*chassis_length} ${y_reflect*(chassis_width/2+wheel_height/2)} 0"
+                rpy="0 0 0" />
+            <axis xyz="0 1 0" />
+        </joint>
+    </xacro:macro>
+    <xacro:wheel x_position="front" y_position="right" x_reflect="1" y_reflect="1" />
+    <xacro:wheel x_position="front" y_position="left" x_reflect="1" y_reflect="-1" />
+    <xacro:wheel x_position="rare" y_position="right" x_reflect="-1" y_reflect="1" />
+    <xacro:wheel x_position="rare" y_position="left" x_reflect="-1" y_reflect="-1" />
 </robot>
